File: BackEnd/KiCad/BrausteuerungV3.sch (KiCad schematic (older format))
At the start: 16 parts, among them IC1 DS18B20, J1 KHTaster, J2 myPiezzo, J3 Transmitter433MHz, J4 HC-06, P1 Power 9V, P2 Switch, U1 arduino_nano

Commit message: reverted to circuit without spannungsteiler HC06
Parts:
- removed P2: Switch, Resistors_THT:R_Axial_DIN0204_L3.6mm_D1.6mm_P1.90mm_Vertical, symbol CONN_01X02
- removed R5: 2.2K, Resistors_THT:R_Axial_DIN0207_L6.3mm_D2.5mm_P10.16mm_Horizontal, symbol R
- removed R6: 4.7K, Resistors_THT:R_Axial_DIN0207_L6.3mm_D2.5mm_P10.16mm_Horizontal, symbol R
- D1: footprint Resistors_THT:R_Axial_DIN0204_L3.6mm_D1.6mm_P1.90mm_Vertical -> LEDs:LED-3MM; symbol LED-RESCUE-BrausteuerungV3 -> LED
- D2: footprint Resistors_THT:R_Axial_DIN0207_L6.3mm_D2.5mm_P10.16mm_Horizontal -> Resistors_ThroughHole:R_Axial_DIN0207_L6.3mm_D2.5mm_P7.62mm_Horizontal
- P1: value Power 9V -> CONN_01X02; footprint Resistors_THT:R_Axial_DIN0204_L3.6mm_D1.6mm_P1.90mm_Vertical -> LEDs:LED-3MM
- R1, R2, R3, R4: footprint Resistors_THT:R_Axial_DIN0207_L6.3mm_D2.5mm_P10.16mm_Horizontal -> Resistors_ThroughHole:Resistor_Horizontal_RM10mm
Connections:
- net +9V: now also D2.2 (A)
- net at U1.29 ((MOSI)#D11): now also J4.4 (RXD)
Other:
- moved on the sheet: P1
Changed lines of the file:
@@
 EESchema Schematic File Version 2
-LIBS:BrausteuerungV3-rescue
 LIBS:myPiezzo
 LIBS:khtaster
 LIBS:hc-06
+LIBS:BrausteuerungV3-rescue
 LIBS:Transmitter433MHz
 LIBS:DS1820
@@
 F 0 "R4" V 8630 2050 50  0000 C CNN
 F 1 "4,7K" V 8550 2050 50  0000 C CNN
-F 2 "Resistors_THT:R_Axial_DIN0207_L6.3mm_D2.5mm_P10.16mm_Horizontal" V 8480 2050 50  0001 C CNN
+F 2 "Resistors_ThroughHole:Resistor_Horizontal_RM10mm" V 8480 2050 50  0001 C CNN
 F 3 "" H 8550 2050 50  0000 C CNN
 	1    8550 2050
@@
 F 0 "R1" V 6730 3400 50  0000 C CNN
 F 1 "330" V 6650 3400 50  0000 C CNN
-F 2 "Resistors_THT:R_Axial_DIN0207_L6.3mm_D2.5mm_P10.16mm_Horizontal" V 6580 3400 50  0001 C CNN
+F 2 "Resistors_ThroughHole:Resistor_Horizontal_RM10mm" V 6580 3400 50  0001 C CNN
 F 3 "" H 6650 3400 50  0000 C CNN
 	1    6650 3400
@@
 F 0 "R2" V 7330 1600 50  0000 C CNN
 F 1 "47K" V 7250 1600 50  0000 C CNN
-F 2 "Resistors_THT:R_Axial_DIN0207_L6.3mm_D2.5mm_P10.16mm_Horizontal" V 7180 1600 50  0001 C CNN
+F 2 "Resistors_ThroughHole:Resistor_Horizontal_RM10mm" V 7180 1600 50  0001 C CNN
 F 3 "" H 7250 1600 50  0000 C CNN
 	1    7250 1600
@@
 F 0 "R3" V 7780 1600 50  0000 C CNN
 F 1 "150K" V 7700 1600 50  0000 C CNN
-F 2 "Resistors_THT:R_Axial_DIN0207_L6.3mm_D2.5mm_P10.16mm_Horizontal" V 7630 1600 50  0001 C CNN
+F 2 "Resistors_ThroughHole:Resistor_Horizontal_RM10mm" V 7630 1600 50  0001 C CNN
 F 3 "" H 7700 1600 50  0000 C CNN
 	1    7700 1600
@@
 $EndComp
 $Comp
-L LED-RESCUE-BrausteuerungV3 D1
+L LED D1
 U 1 1 5788DA4B
 P 6150 3400
 F 0 "D1" H 6150 3500 50  0000 C CNN
 F 1 "LED" H 6150 3300 50  0000 C CNN
-F 2 "Resistors_THT:R_Axial_DIN0204_L3.6mm_D1.6mm_P1.90mm_Vertical" H 6150 3400 50  0001 C CNN
+F 2 "LEDs:LED-3MM" H 6150 3400 50  0001 C CNN
 F 3 "" H 6150 3400 50  0000 C CNN
 	1    6150 3400
@@
 L +9V #PWR02
 U 1 1 5789049D
-P 6200 1250
-F 0 "#PWR02" H 6200 1100 50  0001 C CNN
-F 1 "+9V" H 6200 1390 50  0000 C CNN
-F 2 "" H 6200 1250 50  0000 C CNN
-F 3 "" H 6200 1250 50  0000 C CNN
-	1    6200 1250
+P 6700 1250
+F 0 "#PWR02" H 6700 1100 50  0001 C CNN
+F 1 "+9V" H 6700 1390 50  0000 C CNN
+F 2 "" H 6700 1250 50  0000 C CNN
+F 3 "" H 6700 1250 50  0000 C CNN
+	1    6700 1250
 	1    0    0    -1
 $EndComp
@@
 	7400 2500 7400 2900
 Wire Wire Line
+	7400 2900 8400 2900
+Wire Wire Line
 	8400 2900 8400 3000
 Wire Wire Line
@@
 L CONN_01X02 P1
 U 1 1 579E1182
-P 5950 1400
-F 0 "P1" H 5950 1550 50  0000 C CNN
-F 1 "Power 9V" V 6050 1400 50  0000 C CNN
-F 2 "Resistors_THT:R_Axial_DIN0204_L3.6mm_D1.6mm_P1.90mm_Vertical" H 5950 1400 50  0001 C CNN
-F 3 "" H 5950 1400 50  0000 C CNN
-	1    5950 1400
+P 6400 1400
+F 0 "P1" H 6400 1550 50  0000 C CNN
+F 1 "CONN_01X02" V 6500 1400 50  0000 C CNN
+F 2 "LEDs:LED-3MM" H 6400 1400 50  0001 C CNN
+F 3 "" H 6400 1400 50  0000 C CNN
+	1    6400 1400
 	-1   0    0    1
 $EndComp
 Wire Wire Line
-	6150 1450 6950 1450
+	6600 1450 6950 1450
 Wire Wire Line
 	6950 1450 6950 4500
@@
 F 0 "D2" H 6850 1450 50  0000 C CNN
 F 1 "1n4001" H 6850 1250 50  0000 C CNN
-F 2 "Resistors_THT:R_Axial_DIN0207_L6.3mm_D2.5mm_P10.16mm_Horizontal" H 6850 1350 50  0001 C CNN
+F 2 "Resistors_ThroughHole:R_Axial_DIN0207_L6.3mm_D2.5mm_P7.62mm_Horizontal" H 6850 1350 50  0001 C CNN
 F 3 "" H 6850 1350 50  0000 C CNN
 	1    6850 1350
@@
 	6600 1350 6700 1350
 Wire Wire Line
+	6700 1350 6700 1250
+Connection ~ 6700 1350
+Wire Wire Line
 	8650 2250 8650 1700
-$Comp
-L R R5
-U 1 1 5A568ECA
-P 7850 2900
-F 0 "R5" V 7930 2900 50  0000 C CNN
-F 1 "2.2K" V 7850 2900 50  0000 C CNN
-F 2 "Resistors_THT:R_Axial_DIN0207_L6.3mm_D2.5mm_P10.16mm_Horizontal" V 7780 2900 50  0001 C CNN
-F 3 "" H 7850 2900 50  0000 C CNN
-	1    7850 2900
-	0    1    1    0
-$EndComp
-Wire Wire Line
-	7400 2900 7700 2900
-Wire Wire Line
-	8000 2900 8400 2900
-$Comp
-L R R6
-U 1 1 5A5691D6
-P 7850 3100
-F 0 "R6" V 7930 3100 50  0000 C CNN
-F 1 "4.7K" V 7850 3100 50  0000 C CNN
-F 2 "Resistors_THT:R_Axial_DIN0207_L6.3mm_D2.5mm_P10.16mm_Horizontal" V 7780 3100 50  0001 C CNN
-F 3 "" H 7850 3100 50  0000 C CNN
-	1    7850 3100
-	0    1    1    0
-$EndComp
-Wire Wire Line
-	8000 3100 8150 3100
-Wire Wire Line
-	8150 3100 8150 2900
-Connection ~ 8150 2900
-Wire Wire Line
-	7700 3100 6950 3100
-Connection ~ 6950 3100
-Wire Wire Line
-	6150 1350 6500 1350
-Wire Wire Line
-	6200 1350 6200 1250
-$Comp
-L CONN_01X02 P2
-U 1 1 5A56A656
-P 6550 1150
-F 0 "P2" H 6550 1300 50  0000 C CNN
-F 1 "Switch" V 6650 1150 50  0000 C CNN
-F 2 "Resistors_THT:R_Axial_DIN0204_L3.6mm_D1.6mm_P1.90mm_Vertical" H 6550 1150 50  0001 C CNN
-F 3 "" H 6550 1150 50  0000 C CNN
-	1    6550 1150
-	0    -1   -1   0
-$EndComp
-Connection ~ 6200 1350
 $EndSCHEMATC

Commit message: some HC-06 need a circuit leveler
Parts:
- added P2: Switch, Resistors_THT:R_Axial_DIN0204_L3.6mm_D1.6mm_P1.90mm_Vertical, symbol CONN_01X02
- added R5: 2.2K, Resistors_THT:R_Axial_DIN0207_L6.3mm_D2.5mm_P10.16mm_Horizontal, symbol R
- added R6: 4.7K, Resistors_THT:R_Axial_DIN0207_L6.3mm_D2.5mm_P10.16mm_Horizontal, symbol R
- D1: footprint LEDs:LED-3MM -> Resistors_THT:R_Axial_DIN0204_L3.6mm_D1.6mm_P1.90mm_Vertical; symbol LED -> LED-RESCUE-BrausteuerungV3
- D2: footprint Resistors_ThroughHole:R_Axial_DIN0207_L6.3mm_D2.5mm_P7.62mm_Horizontal -> Resistors_THT:R_Axial_DIN0207_L6.3mm_D2.5mm_P10.16mm_Horizontal
- P1: value CONN_01X02 -> Power 9V; footprint LEDs:LED-3MM -> Resistors_THT:R_Axial_DIN0204_L3.6mm_D1.6mm_P1.90mm_Vertical
- R1, R2, R3, R4: footprint Resistors_ThroughHole:Resistor_Horizontal_RM10mm -> Resistors_THT:R_Axial_DIN0207_L6.3mm_D2.5mm_P10.16mm_Horizontal
Connections:
- net +9V: now also P2.1 (P1); no longer D2.2 (A)
- net GNDREF: now also R6.2
- net at U1.29 ((MOSI)#D11): now also R5.2; no longer J4.4 (RXD)
- new net: J4.4 (RXD), R5.1, R6.1
- new net: D2.2 (A), P2.2 (P2)
Other:
- moved on the sheet: P1
Changed lines of the file:
@@
 EESchema Schematic File Version 2
+LIBS:BrausteuerungV3-rescue
 LIBS:myPiezzo
 LIBS:khtaster
 LIBS:hc-06
-LIBS:BrausteuerungV3-rescue
 LIBS:Transmitter433MHz
 LIBS:DS1820
@@
 F 0 "R4" V 8630 2050 50  0000 C CNN
 F 1 "4,7K" V 8550 2050 50  0000 C CNN
-F 2 "Resistors_ThroughHole:Resistor_Horizontal_RM10mm" V 8480 2050 50  0001 C CNN
+F 2 "Resistors_THT:R_Axial_DIN0207_L6.3mm_D2.5mm_P10.16mm_Horizontal" V 8480 2050 50  0001 C CNN
 F 3 "" H 8550 2050 50  0000 C CNN
 	1    8550 2050
@@
 F 0 "R1" V 6730 3400 50  0000 C CNN
 F 1 "330" V 6650 3400 50  0000 C CNN
-F 2 "Resistors_ThroughHole:Resistor_Horizontal_RM10mm" V 6580 3400 50  0001 C CNN
+F 2 "Resistors_THT:R_Axial_DIN0207_L6.3mm_D2.5mm_P10.16mm_Horizontal" V 6580 3400 50  0001 C CNN
 F 3 "" H 6650 3400 50  0000 C CNN
 	1    6650 3400
@@
 F 0 "R2" V 7330 1600 50  0000 C CNN
 F 1 "47K" V 7250 1600 50  0000 C CNN
-F 2 "Resistors_ThroughHole:Resistor_Horizontal_RM10mm" V 7180 1600 50  0001 C CNN
+F 2 "Resistors_THT:R_Axial_DIN0207_L6.3mm_D2.5mm_P10.16mm_Horizontal" V 7180 1600 50  0001 C CNN
 F 3 "" H 7250 1600 50  0000 C CNN
 	1    7250 1600
@@
 F 0 "R3" V 7780 1600 50  0000 C CNN
 F 1 "150K" V 7700 1600 50  0000 C CNN
-F 2 "Resistors_ThroughHole:Resistor_Horizontal_RM10mm" V 7630 1600 50  0001 C CNN
+F 2 "Resistors_THT:R_Axial_DIN0207_L6.3mm_D2.5mm_P10.16mm_Horizontal" V 7630 1600 50  0001 C CNN
 F 3 "" H 7700 1600 50  0000 C CNN
 	1    7700 1600
@@
 $EndComp
 $Comp
-L LED D1
+L LED-RESCUE-BrausteuerungV3 D1
 U 1 1 5788DA4B
 P 6150 3400
 F 0 "D1" H 6150 3500 50  0000 C CNN
 F 1 "LED" H 6150 3300 50  0000 C CNN
-F 2 "LEDs:LED-3MM" H 6150 3400 50  0001 C CNN
+F 2 "Resistors_THT:R_Axial_DIN0204_L3.6mm_D1.6mm_P1.90mm_Vertical" H 6150 3400 50  0001 C CNN
 F 3 "" H 6150 3400 50  0000 C CNN
 	1    6150 3400
@@
 L +9V #PWR02
 U 1 1 5789049D
-P 6700 1250
-F 0 "#PWR02" H 6700 1100 50  0001 C CNN
-F 1 "+9V" H 6700 1390 50  0000 C CNN
-F 2 "" H 6700 1250 50  0000 C CNN
-F 3 "" H 6700 1250 50  0000 C CNN
-	1    6700 1250
+P 6200 1250
+F 0 "#PWR02" H 6200 1100 50  0001 C CNN
+F 1 "+9V" H 6200 1390 50  0000 C CNN
+F 2 "" H 6200 1250 50  0000 C CNN
+F 3 "" H 6200 1250 50  0000 C CNN
+	1    6200 1250
 	1    0    0    -1
 $EndComp
@@
 	7400 2500 7400 2900
 Wire Wire Line
-	7400 2900 8400 2900
-Wire Wire Line
 	8400 2900 8400 3000
 Wire Wire Line
@@
 L CONN_01X02 P1
 U 1 1 579E1182
-P 6400 1400
-F 0 "P1" H 6400 1550 50  0000 C CNN
-F 1 "CONN_01X02" V 6500 1400 50  0000 C CNN
-F 2 "LEDs:LED-3MM" H 6400 1400 50  0001 C CNN
-F 3 "" H 6400 1400 50  0000 C CNN
-	1    6400 1400
+P 5950 1400
+F 0 "P1" H 5950 1550 50  0000 C CNN
+F 1 "Power 9V" V 6050 1400 50  0000 C CNN
+F 2 "Resistors_THT:R_Axial_DIN0204_L3.6mm_D1.6mm_P1.90mm_Vertical" H 5950 1400 50  0001 C CNN
+F 3 "" H 5950 1400 50  0000 C CNN
+	1    5950 1400
 	-1   0    0    1
 $EndComp
 Wire Wire Line
-	6600 1450 6950 1450
+	6150 1450 6950 1450
 Wire Wire Line
 	6950 1450 6950 4500
@@
 F 0 "D2" H 6850 1450 50  0000 C CNN
 F 1 "1n4001" H 6850 1250 50  0000 C CNN
-F 2 "Resistors_ThroughHole:R_Axial_DIN0207_L6.3mm_D2.5mm_P7.62mm_Horizontal" H 6850 1350 50  0001 C CNN
+F 2 "Resistors_THT:R_Axial_DIN0207_L6.3mm_D2.5mm_P10.16mm_Horizontal" H 6850 1350 50  0001 C CNN
 F 3 "" H 6850 1350 50  0000 C CNN
 	1    6850 1350
@@
 	6600 1350 6700 1350
 Wire Wire Line
-	6700 1350 6700 1250
-Connection ~ 6700 1350
-Wire Wire Line
 	8650 2250 8650 1700
+$Comp
+L R R5
+U 1 1 5A568ECA
+P 7850 2900
+F 0 "R5" V 7930 2900 50  0000 C CNN
+F 1 "2.2K" V 7850 2900 50  0000 C CNN
+F 2 "Resistors_THT:R_Axial_DIN0207_L6.3mm_D2.5mm_P10.16mm_Horizontal" V 7780 2900 50  0001 C CNN
+F 3 "" H 7850 2900 50  0000 C CNN
+	1    7850 2900
+	0    1    1    0
+$EndComp
+Wire Wire Line
+	7400 2900 7700 2900
+Wire Wire Line
+	8000 2900 8400 2900
+$Comp
+L R R6
+U 1 1 5A5691D6
+P 7850 3100
+F 0 "R6" V 7930 3100 50  0000 C CNN
+F 1 "4.7K" V 7850 3100 50  0000 C CNN
+F 2 "Resistors_THT:R_Axial_DIN0207_L6.3mm_D2.5mm_P10.16mm_Horizontal" V 7780 3100 50  0001 C CNN
+F 3 "" H 7850 3100 50  0000 C CNN
+	1    7850 3100
+	0    1    1    0
+$EndComp
+Wire Wire Line
+	8000 3100 8150 3100
+Wire Wire Line
+	8150 3100 8150 2900
+Connection ~ 8150 2900
+Wire Wire Line
+	7700 3100 6950 3100
+Connection ~ 6950 3100
+Wire Wire Line
+	6150 1350 6500 1350
+Wire Wire Line
+	6200 1350 6200 1250
+$Comp
+L CONN_01X02 P2
+U 1 1 5A56A656
+P 6550 1150
+F 0 "P2" H 6550 1300 50  0000 C CNN
+F 1 "Switch" V 6650 1150 50  0000 C CNN
+F 2 "Resistors_THT:R_Axial_DIN0204_L3.6mm_D1.6mm_P1.90mm_Vertical" H 6550 1150 50  0001 C CNN
+F 3 "" H 6550 1150 50  0000 C CNN
+	1    6550 1150
+	0    -1   -1   0
+$EndComp
+Connection ~ 6200 1350
 $EndSCHEMATC
